File: audio-board/rev2/seed3-carrier.kicad_sch (KiCad schematic)
At the start: 51 parts, among them J1 NRJ4HF, J2 SJ3-35063AG, J3 DISPLAY_UART, J4 SJ3-35063AG, J5 NRJ4HF, J6 LINE_OUT, J7 POWER_BOARD, Q1 AO3401A, Q2 2N7002, U1 TLV9061IDBVR, U2 TPA6132A2RTE

Commit message: Set R5 to 3.3k and run U2 at -6 dB
R5 at 100k left the AUX level to the Daisy's unpublished input
impedance: with no module load a 2 Vrms source would reach ~5.4 Vpp,
past the pin's absolute maximum. At 3.3k, R3||R4 into R5 alone caps it
at 2.25 Vpp, and the expected level is 1.5-1.7 Vpp.

At 0 dB, full scale (~0.75 Vrms) clips U2 into 16 ohm headphones: its
1% THD limit there is 25 mW (~0.63 Vrms). Tying G0 to GND gives -6 dB
and ~0.40 Vrms full scale, with 4-6 dB of margin at 16-32 ohm.

DESIGN.md, CHANGES.md, TEST_PLAN.md and the sheet notes carry the new
levels and corners.

Co-Authored-By: Claude Opus 5.5 <noreply@anthropic.com>
Parts:
- R5: value 100k -> 3.3k; LCSC C17900 -> C26032
Connections:
- net +5V: no longer U2.6 (G0)
- net GND: now also U2.6 (G0)
Other:
- note added: "Mono to both channels, 16–64 Ω headphones. R10/C9: ≈ 60 kHz low-pass for DAC noise. U2: TPA6132A2 DirectPath, −6 dB inverting (G0, G1 low): full scale ≈ 0.40 Vrms, no clipping at 16 Ω. Outputs sit at 0 V: no output caps. C10/C11 with U2's 26.4 kΩ inputs: 1.3 Hz high-pass. EN tied to +5V: always on. Layout: run SGND straight to the J4 sleeve. HPVDD/HPVSS are made inside U2: caps only."
- note added: "Passive stereo-to-mono sum straight into AUDIO_IN_2. The Seed3 input is AC-coupled (≈ 5 kΩ): no buffer or coupling cap needed. R5 sets the level (≤ −8 dB even with no Daisy load) and is the source's DC return. C3: RF filter (≈ 110 kHz)."
- note removed: "Mono to both channels, 16–64 Ω headphones. R10/C9: ≈ 64 kHz low-pass for DAC noise. U2: TPA6132A2 DirectPath, 0 dB inverting (G0 high, G1 low). Outputs sit at 0 V: no output caps. C10/C11 with U2's 19.8 kΩ inputs: 1.7 Hz high-pass. EN tied to +5V: always on. Layout: run SGND straight to the J4 sleeve. HPVDD/HPVSS are made inside U2: caps only."
- note removed: "Passive stereo-to-mono sum straight into AUDIO_IN_2. The Seed3 input is AC-coupled (≈ 5 kΩ): no buffer or coupling cap needed. R5 is the source's DC return. C3: RF filter (≈ 65 kHz)."
Changed lines of the file:
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@@
 	)
 	(junction
-		(at 360.68 45.72)
-		(diameter 0)
-		(color 0 0 0 0)
-	)
-	(junction
 		(at 231.14 162.56)
 		(diameter 0)
@@
 	(wire
 		(pts
-			(xy 358.14 48.26) (xy 358.14 45.72)
-		)
-		(stroke
-			(width 0)
-			(type default)
-		)
-	)
-	(wire
-		(pts
 			(xy 386.08 146.05) (xy 386.08 153.67)
 		)
@@
 	(wire
 		(pts
-			(xy 360.68 48.26) (xy 360.68 45.72)
+			(xy 360.68 48.26) (xy 360.68 40.64)
 		)
 		(stroke
@@
 	(wire
 		(pts
-			(xy 358.14 45.72) (xy 360.68 45.72)
-		)
-		(stroke
-			(width 0)
-			(type default)
-		)
-	)
-	(wire
-		(pts
 			(xy 22.86 134.62) (xy 22.86 139.7)
 		)
@@
 	(wire
 		(pts
-			(xy 360.68 45.72) (xy 360.68 40.64)
-		)
-		(stroke
-			(width 0)
-			(type default)
-		)
-	)
-	(wire
-		(pts
 			(xy 175.26 241.3) (xy 177.8 241.3)
 		)
@@
 		)
 	)
-	(text "Passive stereo-to-mono sum\nstraight into AUDIO_IN_2. The Seed3\ninput is AC-coupled (≈ 5 kΩ): no\nbuffer or coupling cap needed.\nR5 is the source's DC return.\nC3: RF filter (≈ 65 kHz)."
+	(text "Passive stereo-to-mono sum\nstraight into AUDIO_IN_2. The Seed3\ninput is AC-coupled (≈ 5 kΩ): no\nbuffer or coupling cap needed.\nR5 sets the level (≤ −8 dB even\nwith no Daisy load) and is the\nsource's DC return.\nC3: RF filter (≈ 110 kHz)."
 		(exclude_from_sim no)
 		(at 93.98 81.28 0)
@@
 		)
 	)
-	(text "Mono to both channels, 16–64 Ω headphones. R10/C9: ≈ 64 kHz low-pass for DAC noise.\nU2: TPA6132A2 DirectPath, 0 dB inverting (G0 high, G1 low). Outputs sit at 0 V: no output caps.\nC10/C11 with U2's 19.8 kΩ inputs: 1.7 Hz high-pass. EN tied to +5V: always on.\nLayout: run SGND straight to the J4 sleeve. HPVDD/HPVSS are made inside U2: caps only."
+	(text "Mono to both channels, 16–64 Ω headphones. R10/C9: ≈ 60 kHz low-pass for DAC noise.\nU2: TPA6132A2 DirectPath, −6 dB inverting (G0, G1 low): full scale ≈ 0.40 Vrms, no clipping at 16 Ω.\nOutputs sit at 0 V: no output caps. C10/C11 with U2's 26.4 kΩ inputs: 1.3 Hz high-pass. EN tied to +5V: always on.\nLayout: run SGND straight to the J4 sleeve. HPVDD/HPVSS are made inside U2: caps only."
 		(exclude_from_sim no)
 		(at 271.78 91.44 0)
@@
 		)
 	)
+	(wire
+		(pts
+			(xy 358.14 48.26) (xy 358.14 45.72)
+		)
+		(stroke
+			(width 0)
+			(type default)
+		)
+	)
+	(wire
+		(pts
+			(xy 358.14 45.72) (xy 349.25 45.72)
+		)
+		(stroke
+			(width 0)
+			(type default)
+		)
+	)
+	(junction
+		(at 349.25 45.72)
+		(diameter 0)
+		(color 0 0 0 0)
+	)
 	(symbol
 		(lib_id "power:GND")
@@
 			)
 		)
-		(property "Value" "100k"
+		(property "Value" "3.3k"
 			(at 66.04 96.52 0)
 			(show_name no)
@@
 			)
 		)
-		(property "LCSC" "C17900"
+		(property "LCSC" "C26032"
 			(at 68.58 95.25 0)
 			(hide yes)

Commit message: Add a pad after the guitar buffer for active pickups
U1 at unity gain could swing ~4.8 Vpp into AUDIO_IN_1, past the Daisy
pin's 3.6 Vpp full scale and +-1.8 V absolute maximum. R20 (470 ohm,
C4502) into R21 (1k to GND, C4410) scales U1's swing so the pin never
sees more than 3.4 Vpp, even with no module load and U1 at both rails.

The input is now clean to ~4.8 Vpp at J1, which covers passive and
typical 9 V active pickups; hotter sources clip harmlessly in U1.
Passive pickups lose 3.9 dB of converter signal-to-noise. R20/R21 sit
above U1 pin 1 on the board.

DESIGN.md, TEST_PLAN.md (new 1.21b and 5.19), CHANGES.md and the sheet
note are updated. One more extended part (C4502).

Co-Authored-By: Claude Opus 5.5 <noreply@anthropic.com>
Parts:
- added R20: 470, Resistor_SMD:R_1206_3216Metric_Pad1.30x1.75mm_HandSolder, symbol Device:R_Small_US
- added R21: 1k, Resistor_SMD:R_1206_3216Metric_Pad1.30x1.75mm_HandSolder, symbol Device:R_Small_US
Connections:
- net AUDIO_IN_1: now also R20.2, R21.1; no longer U1.1, U1.4 (-)
- net GND: now also R21.2
- new net: R20.1, U1.1, U1.4 (-)
Other:
- note added: "R1 (1 MΩ to VREF) sets the guitar load and the DC bias. U1A is a unity-gain buffer: input trim is in firmware. R20/R21 pad: U1's swing (≤ 4.8 Vpp clean) reaches the Daisy at ≤ 3.4 Vpp, so no pickup can overdrive it. J1's tip switch shorts the input to GND with no plug in. C1 is an RF shunt. R2 protects U1A's input."
- note removed: "R1 (1 MΩ to VREF) sets the guitar load and the DC bias. U1A is a unity-gain buffer: input trim is in firmware. J1's tip switch shorts the input to GND with no plug in. C1 is an RF shunt. R2 protects U1A's input."

Commit message: Lower the line-out impedance: R11 to 1k, C16 to 3.3 nF
R11 is the line out's output impedance. At 3.3k it cost 2.7 dB into a
10k input and more into lower-impedance gear. At 1k it costs 0.9 dB,
and a shorted J5 still leaves the Daisy at 1k, above its 600 ohm
minimum load. C16 goes to 3.3 nF to keep the 48 kHz corner.

R11 reuses the basic 1k (C4410). JLC had no 3.3 nF C0G 1206 in stock,
so C16 is the 0805 FH 0805CG332J500NT (C486355, extended), placed
where the 1206 was. DESIGN.md, TEST_PLAN.md, CHANGES.md and the sheet
note carry the new values.

Co-Authored-By: Claude Opus 5.5 <noreply@anthropic.com>
Parts:
- C16: value 1nF -> 3.3nF; footprint Capacitor_SMD:C_1206_3216Metric_Pad1.33x1.80mm_HandSolder -> Capacitor_SMD:C_0805_2012Metric_Pad1.18x1.45mm_HandSolder; LCSC C1885 -> C486355
- R11: value 3.3k -> 1k; LCSC C26032 -> C4410
Other:
- note added: "AUDIO_OUT_2 drives J5 (external) and J6 (speaker amp) directly. R11/C16: ≈ 48 kHz low-pass, 1k out. R12: DC return. With headphones in, the firmware drives SPK_EN low. J5 stays live."
- note removed: "AUDIO_OUT_2 drives J5 (external) and J6 (speaker amp) directly. R11/C16: ≈ 48 kHz low-pass. R12: DC return. With headphones in, the firmware drives SPK_EN low. J5 stays live."
Changed lines of the file:
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@@
 		)
 	)
-	(text "AUDIO_OUT_2 drives J5 (external) and J6 (speaker amp)\ndirectly. R11/C16: ≈ 48 kHz low-pass. R12: DC return.\nWith headphones in, the firmware drives SPK_EN low.\nJ5 stays live."
+	(text "AUDIO_OUT_2 drives J5 (external) and J6 (speaker amp)\ndirectly. R11/C16: ≈ 48 kHz low-pass, 1k out. R12: DC return.\nWith headphones in, the firmware drives SPK_EN low.\nJ5 stays live."
 		(exclude_from_sim no)
 		(at 271.78 191.77 0)
@@
 			)
 		)
-		(property "Value" "1nF"
+		(property "Value" "3.3nF"
 			(at 302.26 182.88 0)
 			(show_name no)
@@
 			)
 		)
-		(property "Footprint" "Capacitor_SMD:C_1206_3216Metric_Pad1.33x1.80mm_HandSolder"
+		(property "Footprint" "Capacitor_SMD:C_0805_2012Metric_Pad1.18x1.45mm_HandSolder"
 			(at 299.72 181.61 0)
 			(hide yes)
@@
 			)
 		)
-		(property "LCSC" "C1885"
+		(property "LCSC" "C486355"
 			(at 299.72 181.61 0)
 			(hide yes)
@@
 			)
 		)
-		(property "Value" "3.3k"
+		(property "Value" "1k"
 			(at 292.1 175.26 90)
 			(show_name no)
@@
 			)
 		)
-		(property "LCSC" "C26032"
+		(property "LCSC" "C4410"
 			(at 292.1 179.07 0)
 			(hide yes)

Commit message: Add a 0 ohm jumper in the line out as a DC-block option
The line out has no coupling cap and assumes Daisy pin 19 sits at 0 V
DC, which TEST_PLAN 5.16 has yet to confirm. R22 (0 ohm, C17888, basic)
now sits between the R11/C16 filter and LINE_OUT. If the pin carries
DC, R22 is swapped for a 10 uF 1206 ceramic without a respin; R12 then
holds LINE_OUT at 0 V and the corner with a 10k load is ~1.8 Hz.

R22 sits below R11, left of R12, on the board. DESIGN.md, TEST_PLAN.md,
CHANGES.md and the sheet note point at R22 instead of "fit a cap".

Co-Authored-By: Claude Opus 5.5 <noreply@anthropic.com>
Parts:
- added R22: 0, Resistor_SMD:R_1206_3216Metric_Pad1.30x1.75mm_HandSolder, symbol Device:R_Small_US
Connections:
- net LINE_OUT: now also R22.2; no longer C16.1, R11.2
- new net: C16.1, R11.2, R22.1
Other:
- note added: "AUDIO_OUT_2 drives J5 (external) and J6 (speaker amp) directly. R11/C16: ≈ 48 kHz low-pass, 1k out. R12: DC return. R22: 0 Ω; fit 10 µF if pin 19 has DC (TEST_PLAN 5.16). With headphones in, the firmware drives SPK_EN low. J5 stays live."
- note removed: "AUDIO_OUT_2 drives J5 (external) and J6 (speaker amp) directly. R11/C16: ≈ 48 kHz low-pass, 1k out. R12: DC return. With headphones in, the firmware drives SPK_EN low. J5 stays live."
Changed lines of the file:
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@@
 		)
 	)
-	(wire
-		(pts
-			(xy 299.72 179.07) (xy 312.42 179.07)
-		)
-		(stroke
-			(width 0)
-			(type default)
-		)
-	)
 	(label "LINE_OUT"
-		(at 312.42 179.07 0)
+		(at 317.5 179.07 0)
 		(effects
 			(font
@@
 		)
 	)
-	(text "AUDIO_OUT_2 drives J5 (external) and J6 (speaker amp)\ndirectly. R11/C16: ≈ 48 kHz low-pass, 1k out. R12: DC return.\nWith headphones in, the firmware drives SPK_EN low.\nJ5 stays live."
+	(text "AUDIO_OUT_2 drives J5 (external) and J6 (speaker amp)\ndirectly. R11/C16: ≈ 48 kHz low-pass, 1k out. R12: DC return.\nR22: 0 Ω; fit 10 µF if pin 19 has DC (TEST_PLAN 5.16).\nWith headphones in, the firmware drives SPK_EN low.\nJ5 stays live."
 		(exclude_from_sim no)
 		(at 271.78 191.77 0)
@@
 		(color 0 0 0 0)
 	)
+	(wire
+		(pts
+			(xy 299.72 179.07) (xy 304.8 179.07)
+		)
+		(stroke
+			(width 0)
+			(type default)
+		)
+	)
+	(wire
+		(pts
+			(xy 309.88 179.07) (xy 317.5 179.07)
+		)
+		(stroke
+			(width 0)
+			(type default)
+		)
+	)
 	(symbol
 		(lib_id "power:GND")
@@
 					(unit 1)
 				)
+			)
+		)
+	)
+	(symbol
+		(lib_id "Device:R_Small_US")
+		(at 307.34 179.07 90)
+		(unit 1)
+		(body_style 1)
+		(exclude_from_sim no)
+		(in_bom yes)
+		(on_board yes)
+		(in_pos_files yes)
+		(dnp no)
+		(property "Reference" "R22"
+			(at 307.34 172.72 90)
+			(show_name no)
+			(do_not_autoplace no)
+			(effects
+				(font
+					(size 1.27 1.27)
+				)
+			)
+		)
+		(property "Value" "0"
+			(at 307.34 175.26 90)
+			(show_name no)
+			(do_not_autoplace no)
+			(effects
+				(font
+					(size 1.27 1.27)
+				)
+			)
+		)
+		(property "Footprint" "Resistor_SMD:R_1206_3216Metric_Pad1.30x1.75mm_HandSolder"
+			(at 307.34 179.07 0)
+			(hide yes)
+			(show_name no)
+			(do_not_autoplace no)
+			(effects
+				(font
+					(size 1.27 1.27)
+				)
+			)
+		)
+		(property "Datasheet" ""
+			(at 307.34 179.07 0)
+			(hide yes)
+			(show_name no)
+			(do_not_autoplace no)
+			(effects
+				(font
+					(size 1.27 1.27)
+				)
+			)
+		)
+		(property "Description" "Resistor, small US symbol"
+			(at 307.34 179.07 0)
+			(hide yes)
+			(show_name no)
+			(do_not_autoplace no)
+			(effects
+				(font
+					(size 1.27 1.27)
+				)
+			)
+		)
+		(property "LCSC" "C17888"
+			(at 307.34 179.07 0)
+			(hide yes)
+			(show_name no)
+			(do_not_autoplace no)
+			(effects
+				(font
+					(size 1.27 1.27)
+				)
+			)
+		)
+		(pin "1"
+		)
+		(pin "2"
+		)
+		(instances
+			(project "seed3-carrier"
+				(path "/94ecceca-f8ce-4e68-9c84-99ac5115dfb9"
+					(reference "R22")
+					(unit 1)
+				)

Commit message: Add ESD diodes on every jack signal contact
D1-D6 (Nexperia PESD5V0S1BA, SOD-323, C19224) clamp J1 tip, J2
tip/ring, J4 tip/ring and J5 tip to GND, each placed beside its jack.
Bidirectional with a 5 V working voltage, so no audio signal on these
contacts reaches it; 5 nA leakage and 35 pF don't load the 1 MOhm
guitar input. The isolated J2/J4 detect switches need none.

The sheet gains a JACK ESD PROTECTION section, with the power-board
block shifted left to make room, and the J1/J2 nets are named
GTR_TIP, AUX_TIP and AUX_RING. DESIGN.md also records that the J2/J4
footprint matches the Same Sky datasheet layout; TEST_PLAN adds 1.21c.

Co-Authored-By: Claude Opus 5.5 <noreply@anthropic.com>
Parts:
- added D1, D2, D3, D4, D5, D6: PESD5V0S1BA, Diode_SMD:D_SOD-323, symbol Device:D_TVS
Connections:
- net GND: now also D1.1 (A1), D2.1 (A1), D3.1 (A1), D4.1 (A1), D5.1 (A1), D6.1 (A1)
- net HP_L: now also D4.2 (A2)
- net HP_R: now also D5.2 (A2)
- net LINE_OUT: now also D6.2 (A2)
- net GTR_TIP: now reaches C1.1, C2.1, J1.T
- net GTR_TIP: now also D1.2 (A2)
- net AUX_RING: now reaches J2.2 (R), R4.1
- net AUX_RING: now also D3.2 (A2)
- net AUX_TIP: now reaches J2.3 (T), R3.1
- net AUX_TIP: now also D2.2 (A2)
Other:
- note added: "D1–D6: bidirectional ESD diodes (PESD5V0S1BA: 5 V working, 35 pF, 5 nA) from every jack signal contact to GND, each placed at its jack. Guitar signals stay below the 5 V working voltage. The J2/J4 detect switches are isolated from the plug: no diode."
- note added: "JACK ESD PROTECTION"
- moved on the sheet: C17, C18, J7, Q2, R13, R14, R15, R16, R17

Commit message: Drop the 1/4" line out, the input pad, R22 and D6
The speaker send now goes only to the internal header (J5, was J6), and the
power board connector is J6 (was J7). R20 stays as a 470 ohm series resistor
with no pad, since active pickups are out of scope. Docs and test plan follow.

Co-Authored-By: Claude Opus 5.5 <noreply@anthropic.com>
Parts:
- removed D6: PESD5V0S1BA, Diode_SMD:D_SOD-323, symbol Device:D_TVS
- removed J5: NRJ4HF, Connector_Audio:Jack_6.35mm_Neutrik_NRJ4HF_Horizontal, symbol Connector_Audio:AudioJack2
- removed R21: 1k, Resistor_SMD:R_1206_3216Metric_Pad1.30x1.75mm_HandSolder, symbol Device:R_Small_US
- removed R22: 0, Resistor_SMD:R_1206_3216Metric_Pad1.30x1.75mm_HandSolder, symbol Device:R_Small_US
- C1: footprint Capacitor_SMD:C_1206_3216Metric_Pad1.33x1.80mm_HandSolder -> Capacitor_SMD:C_0805_2012Metric_Pad1.18x1.45mm_HandSolder; LCSC C107179 -> C1790
- C10, C11: footprint Capacitor_SMD:C_1210_3225Metric_Pad1.33x2.70mm_HandSolder -> Capacitor_SMD:C_0805_2012Metric_Pad1.18x1.45mm_HandSolder; LCSC C86052 -> C1779; MPN GRM32ER71H475KA88L -> CL21A475KAQNNNE
- R10, R5: footprint Resistor_SMD:R_1206_3216Metric_Pad1.30x1.75mm_HandSolder -> Resistor_SMD:R_0805_2012Metric_Pad1.20x1.40mm_HandSolder; LCSC C26032 -> C26010
- R20: footprint Resistor_SMD:R_1206_3216Metric_Pad1.30x1.75mm_HandSolder -> Resistor_SMD:R_0805_2012Metric_Pad1.20x1.40mm_HandSolder; LCSC C4502 -> C17710
- renumbered J6 to J5, J7 to J6
Connections:
- net LINE_OUT: now also C16.1, R11.2
Other:
- note added: "AUDIO_OUT_2 drives J5 (to the speaker amp) directly. R11/C16: ≈ 48 kHz low-pass, 1k out. R12: DC return. Assumes pin 19 sits at 0 V DC (TEST_PLAN 5.16). With headphones in, the firmware drives SPK_EN low."
- note added: "D1–D5: bidirectional ESD diodes (PESD5V0S1BA: 5 V working, 35 pF, 5 nA) from every jack signal contact to GND, each placed at its jack. Guitar signals stay below the 5 V working voltage. The J2/J4 detect switches are isolated from the plug: no diode."
- note added: "J6 goes to the power board (JST-XH, 8 pins). Pins 5–7 are 3.3 V logic: nothing above 3.3 V on them. SPK_MUTE is open drain. The power board pulls it up, so the speaker amp stays muted unless SPK_EN is high. R13, R16 and R14 limit current into an unpowered Daisy. R15 holds PWR_HOLD low while the Daisy is absent or booting."
- note added: "Q1: reverse-polarity protection for 5V_IN (J6). C5 (low-ESR) damps the harness ringing. C4 is the entry ceramic."
- note added: "R1 (1 MΩ to VREF) sets the guitar load and the DC bias. U1A is a unity-gain buffer: input trim is in firmware. R20 limits current into the Daisy pin if U1 is ever overdriven. Passive pickups only: no pad. J1's tip switch shorts the input to GND with no plug in. C1 is an RF shunt. R2 protects U1A's input."
- note added: "SPEAKER SEND"
- note removed: "AUDIO_OUT_2 drives J5 (external) and J6 (speaker amp) directly. R11/C16: ≈ 48 kHz low-pass, 1k out. R12: DC return. R22: 0 Ω; fit 10 µF if pin 19 has DC (TEST_PLAN 5.16). With headphones in, the firmware drives SPK_EN low. J5 stays live."
- note removed: "D1–D6: bidirectional ESD diodes (PESD5V0S1BA: 5 V working, 35 pF, 5 nA) from every jack signal contact to GND, each placed at its jack. Guitar signals stay below the 5 V working voltage. The J2/J4 detect switches are isolated from the plug: no diode."
- note removed: "J7 goes to the power board (JST-XH, 8 pins). Pins 5–7 are 3.3 V logic: nothing above 3.3 V on them. SPK_MUTE is open drain. The power board pulls it up, so the speaker amp stays muted unless SPK_EN is high. R13, R16 and R14 limit current into an unpowered Daisy. R15 holds PWR_HOLD low while the Daisy is absent or booting."
- note removed: "LINE OUT & SPEAKER SEND"
- note removed: "Q1: reverse-polarity protection for 5V_IN (J7). C5 (low-ESR) damps the harness ringing. C4 is the entry ceramic."
- note removed: "R1 (1 MΩ to VREF) sets the guitar load and the DC bias. U1A is a unity-gain buffer: input trim is in firmware. R20/R21 pad: U1's swing (≤ 4.8 Vpp clean) reaches the Daisy at ≤ 3.4 Vpp, so no pickup can overdrive it. J1's tip switch shorts the input to GND with no plug in. C1 is an RF shunt. R2 protects U1A's input."
